File: ServoShield.kicad_pcb (KiCad board)
At the start: 2 copper layers, 68.6 x 53.3 mm, 54 parts, among them P1 M03, P10 M03, P11 M03, P12 M03, P13 M03, P14 M03, P15 M03, P16 M03, P2 M03, P3 M03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

Commit message: Completed v1.0
Parts:
- added LOGO_FREETRONICS_SMALL: val**, FT:LOGO_FREETRONICS_MIDSIZE, F.Cu at (178.8, 46.9)
- added LOGO_GND_SILKSCREEN: VAL**, FT:LOGO_GND_SILKSCREEN, F.Cu at (197.4, 95.2)
- added LOGO_GND_SILKSCREEN: VAL**, FT:LOGO_GND_SILKSCREEN, F.Cu at (231.1, 54.1)
- added LOGO_GND_SILKSCREEN: VAL**, FT:LOGO_GND_SILKSCREEN, F.Cu at (231.1, 87.2)
- C1, C5: footprint Capacitors_SMD:c_1210 -> FT:1210
- C7: footprint Capacitors_SMD:C_0402 -> FT:SM0603_Capa
- L1: footprint FT:SRU1038_IND -> FT:CDRH125
- R9: value 14k -> 8K
- moved SJ1 6.93 mm to (186.9, 55.2), turned to 0 degrees
- moved Q2 6.27 mm to (185.4, 50.7)
- moved R7 5.35 mm to (197.0, 84.0), turned to 135 degrees
- moved R2 4.48 mm to (182.0, 51.2)
- moved C5 2.56 mm to (208.0, 66.1), turned to 270 degrees
- moved Q1 1.93 mm to (185.5, 53.2)
- moved L1 1.22 mm to (198.2, 60.6), turned to 90 degrees
- moved D1 0.80 mm to (189.2, 71.0)
- moved R3 0.50 mm to (221.0, 69.9)
- moved SJ7 0.30 mm to (186.9, 52.2)
- moved R1 0.30 mm to (221.0, 73.9)
- moved P13 0.20 mm to (187.8, 90.2)
- moved P16 0.20 mm to (195.4, 90.2)
- moved C7 0.20 mm to (202.3, 68.9)
- moved P14 0.20 mm to (190.3, 90.2)
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Connections:
- R2 pad 2: /SCL_IO -> /SDA_IO
- R2 pad 4: /SCL_PWM -> /SDA_PWM
- R2 pad 6: /SDA_IO -> /SCL_IO
- R2 pad 8: /SDA_PWM -> /SCL_PWM
Routing:
- net GND: track 53.1 -> 148.7 mm, vias 22 -> 36
- net /A5_SCL: track 104.1 -> 124.6 mm
- net /A4_SDA: track 102.5 -> 120.7 mm
- net +5V: track 113.5 -> 123.7 mm, vias 4 -> 3
- net /SCL_PWM: track 55.8 -> 65.0 mm, vias 4 -> 6
- net /PWM14: track 22.2 -> 16.1 mm
- net IORef: track 79.3 -> 85.3 mm, vias 3 -> 1
- net Net-(P13-Pad1): track 5.85 -> 11.5 mm
- net /PWM15: track 20.8 -> 15.5 mm
- net /PWM13: track 23.2 -> 18.2 mm
- net /PWM12: track 24.5 -> 20.1 mm
- net +6V: track 24.9 -> 21.4 mm
- net Net-(P14-Pad1): track 5.13 -> 8.41 mm
- net /SDA_PWM: track 55.7 -> 58.1 mm
- net /SCL_IO: track 18.2 -> 16.2 mm
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Other:
- board text added: "+"
- board text added: "+5V"
- board text added: "+5V/IORef"
- board text added: "+6V"
- board text added: "14"
- board text added: "15"
- board text added: "Brown Black Black"
- board text added: "Close all 3 Jumpers for Pre-R3 Boards"
- board text added: "Copyright (C) 2014 Freetronics Pty Ltd TAPR Open Hardware License Designed by Angus Gratton"
- board text added: "D10/~OE"
- board text added: "Default I2C Address 0x40"
- board text added: "I2C Address Selection Default 0x40, Available 0x40-0x4F"
- board text added: "JR Futaba Hitec"
- board text added: "Orange White Yellow"
- board text added: "RESET"
- board text added: "Red Red Red"
- board text added: "SCL/A5"
- board text added: "SDA/A4"
- board text added: "SIG"
- board text added: "SKU: SERV"
- board text added: "Servo Pinouts"
- board text added: "ServoShield"
- board text added: "Signal"
- board text added: "V1.0"
- board text added: "VCC"
- board text added: "VCC Select"
- board text added: "tron.cc/serv"

Commit message: Small tweaks
Parts:
- C1, C5: value 10uF -> 10uF 10V
- C2: value 68uF 25V -> 68uF 10V
- C3, C7: value 1uF -> 1uF 25V
- D1: value B540C -> B340 40V 3A
Connections:
- SHIELD1 pad SP1: Net-(SHIELD1-PadSP1) -> (no net)
- SHIELD1 pad SP2: Net-(SHIELD1-PadSP2) -> (no net)
- SHIELD1 pad SP3: Net-(SHIELD1-PadSP3) -> (no net)
- SHIELD1 pad SP4: Net-(SHIELD1-PadSP4) -> (no net)
- SHIELD1 pad SP5: Net-(SHIELD1-PadSP5) -> (no net)

Commit message: V1.1: Add power LED, fix SSOP footprint for PCA9685
Parts:
- added LED1: LED, FT:LED-0603, F.Cu at (177.2, 52.3)
- added R10: 1K, FT:0603, F.Cu at (177.2, 50.6)
- U1: footprint FT:SSOP28 -> FT:SSOP28-4.4MM
- moved U1 0.21 mm to (213.2, 74.2)
Routing:
- net GND: track 148.7 -> 154.2 mm
- net /SDA_PWM: track 58.1 -> 60.1 mm
- net Net-(LED1-PadA): track 0.00 -> 1.72 mm
- net /PWM12: track 20.1 -> 18.7 mm
- net +5V: track 123.7 -> 125.0 mm
- net /PWM3: track 3.54 -> 4.55 mm
- net /PWM2: track 3.48 -> 4.44 mm
- net /PWM6: track 4.47 -> 5.43 mm
- net /PWM4: track 3.94 -> 4.88 mm
- net /PWM5: track 4.21 -> 5.15 mm
- net /PWM7: track 4.93 -> 5.87 mm
- net Net-(R6-Pad5): track 14.9 -> 15.9 mm
- net Net-(R6-Pad3): track 15.8 -> 16.7 mm
- net Net-(R6-Pad1): track 16.4 -> 17.3 mm
- net /PWM0: track 3.36 -> 4.30 mm
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Other:
- board text added: "Power"
- board text added: "V1.1"
- board text removed: "V1.0"

Commit message: Small V1.1 silkscreen cleanup, new library revision
Parts:
- C2: value 68uF 10V -> 47uF 25V; footprint FT:CAP_ELECTRO_SMT_D -> FT:CAP_ELECTRO_SMD_6.6mm
- C3, C6, C7: footprint FT:SM0603_Capa -> FT:0603_CAP
- C4: footprint FT:CAP_ELECTRO_SMT_D -> FT:CAP_ELECTRO_SMD_6.6mm
- D1: footprint FT:SMC-DIODE -> FT:DIODE_SMC
- L1: footprint FT:CDRH125 -> FT:IND_CDRH125
- Q1, Q2: footprint FT:SOT323_MOSFET -> FT:SOT323_FET
- SW1: footprint FT:TACTILE_SWITCH_SMD_2PIN_TINY -> FT:SW_PUSHBUTTON_TINY_2PIN
- U1: footprint FT:SSOP28-4.4MM -> FT:SSOP28_4mm
- U2: footprint FT:SO08 -> FT:SO08_4mm
- moved C2 0.82 mm to (216.0, 58.0)
- moved SJ1 0.81 mm to (187.0, 56.0)
- moved SJ2 0.51 mm to (186.9, 50.4)
- moved SJ7 0.50 mm to (186.9, 52.7)
- moved C4 0.28 mm to (195.4, 78.4)
Routing:
- net GND: track 154.2 -> 158.1 mm
- net /SCL_PWM: track 65.0 -> 61.5 mm
- net IORef: track 85.3 -> 83.4 mm
- net Net-(JP4-Pad4): track 4.45 -> 6.29 mm
- net +5V: track 125.0 -> 126.6 mm
- net /A5_SCL: track 124.6 -> 125.6 mm
- net Net-(P6-Pad1): track 5.79 -> 4.99 mm
- net /D5: track 4.45 -> 5.08 mm
Other:
- rule pad_to_mask_clearance: 0 -> 0.05
